File: KiCad/MiniTx_Er9XR_PRO.kicad_pcb (KiCad board)
At the start: 2 copper layers, 17.1 x 12.4 mm, 27 parts, among them J1 CONN_01X03, J10 LED2, J3 PWR2, J4 ENABLE2, J5 LED1, J6 LED2, J7 MODULE1_POWER, J8 MODULE2_POWER, J9 LED1, U2 MIC5219-3.3BM5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

Commit message: Not sure how many changes
Parts:
- removed C4: 2.2uf, Capacitors_SMD:C_0603_HandSoldering
- removed R1: 1K, Resistors_SMD:R_0603_HandSoldering
- removed R7: 5K, Resistors_SMD:R_0603_HandSoldering
- removed U3: MIC5219-3.3BM5, TO_SOT_Packages_SMD:SOT-23-5
- added C1: 470, Capacitors_SMD:C_0603_HandSoldering, F.Cu at (134.2, 94.9)
- added C3: 2.2uf, Capacitors_SMD:C_0603_HandSoldering, F.Cu at (137.8, 94.9)
- added C7: 2.2uf, Capacitors_SMD:C_0603_HandSoldering, F.Cu at (131.2, 90.0)
- added J1: CONN_01X03, Connectors:PINHEAD1-3, F.Cu at (128.4, 94.1)
- added J11: CH5, Connectors:PINHEAD1-3, F.Cu at (141.2, 119.1)
- added J11: CH5, Connectors:PINHEAD1-3, F.Cu at (141.2, 105.8)
- added J2: BAT2, Connectors:PINHEAD1-2, F.Cu at (108.8, 117.2)
- added J5: LED1, Connectors:PINHEAD1-2, F.Cu at (141.1, 88.9)
- added J6: THRTL1, Connectors:PINHEAD1-2, F.Cu at (130.2, 120.0)
- added J7: MODULE1_POWER, Connectors:PINHEAD1-2, F.Cu at (141.1, 95.0)
- added J9: LED1, Connectors:PINHEAD1-2, F.Cu at (130.3, 125.3)
- added R2: 300, Resistors_SMD:R_0603_HandSoldering, F.Cu at (137.7, 90.0)
- added R4: 600, Resistors_SMD:R_0603_HandSoldering, F.Cu at (133.2, 121.5)
- added R6: 10K, Resistors_SMD:R_0603_HandSoldering, F.Cu at (137.8, 120.8)
- added R8: 20K, Resistors_SMD:R_0603_HandSoldering, F.Cu at (135.6, 123.3)
- added REF**: Socket_Strip_Straight_1x01_Pitch2.54mm, Socket_Strips:Socket_Strip_Straight_1x01_Pitch2.54mm, F.Cu at (118.0, 110.2)
- added U2: MIC5219-3.3BM5, TO_SOT_Packages_SMD:SOT-23-5, F.Cu at (134.2, 91.2)
- C2: value 470 -> 2.2uf
- J10: value LED2 -> STAB; footprint Connectors:PINHEAD1-2 -> Connectors:PINHEAD1-3
- J3: value PWR2 -> BAT1
- J4: value ENABLE2 -> BAT; footprint Connectors:PINTST -> Connectors:PINHEAD1-2
- J6: value LED2 -> THRTL1
- J8: value MODULE2_POWER -> 3.3V; footprint Connectors:PINHEAD1-2 -> Connectors:PINHEAD1-3
- R3: value 300 -> 30K
- R5: value 600 -> 10K
- moved R3 61.0 mm to (114.6, 112.3)
- moved R5 60.2 mm to (114.6, 115.2), turned to 180 degrees
- moved J10 47.7 mm to (122.6, 111.8), turned to 270 degrees
- moved J4 47.3 mm to (108.8, 106.8), turned to 90 degrees
- moved J3 46.9 mm to (108.8, 111.9), turned to 90 degrees
- moved R4 41.9 mm to (133.2, 108.2), turned to 270 degrees
- moved J6 34.4 mm to (130.2, 106.7), turned to 90 degrees
- moved C2 33.4 mm to (111.8, 105.5), turned to 270 degrees
- moved U4 30.8 mm to (115.6, 105.5)
- moved R8 29.3 mm to (135.6, 110.0), turned to 270 degrees
- moved J8 23.4 mm to (122.6, 109.2), turned to 90 degrees
- moved C5 20.3 mm to (115.7, 108.2), turned to 180 degrees
- moved C6 14.7 mm to (118.9, 105.5), turned to 270 degrees
- moved R6 12.0 mm to (137.8, 107.4), turned to 90 degrees
- moved J9 6.27 mm to (130.2, 112.0), turned to 90 degrees
Connections:
- net CH5 renamed Net-(J11-Pad2)
- C2 pad 1: Net-(C2-Pad1) -> +BATT
- J10 pad 1: GND -> +3V3
- J3 pad 2: Net-(J3-Pad2) -> +BATT
- J4 pad 1: Net-(J4-Pad1) -> GND
- J6 pad 2: GND -> Net-(J11-Pad1)
- J8 pad 1: Net-(C4-Pad1) -> +3V3
- J8 pad 2: GND -> +3V3
- R3 pad 1: Net-(C4-Pad1) -> +BATT
- R3 pad 2: Net-(J6-Pad1) -> Net-(J10-Pad2)
- R4 pad 1: Net-(R4-Pad1) -> Net-(J6-Pad1)
- R5 pad 1: Net-(R5-Pad1) -> Net-(J10-Pad2)
- R5 pad 2: Net-(J10-Pad2) -> GND
- R6 pad 2: Net-(R4-Pad1) -> Net-(J6-Pad1)
Routing:
- net GND: track 14.3 -> 92.4 mm
- net +BATT: track 0.00 -> 32.4 mm
- net Net-(J11-Pad1): track 0.00 -> 23.5 mm
- net Net-(J6-Pad1): track 0.00 -> 16.2 mm
- net +3V3: track 0.00 -> 13.7 mm
- net Net-(J11-Pad2): track 0.00 -> 11.6 mm
- net Net-(J10-Pad2): track 0.00 -> 10.0 mm
- net Net-(C3-Pad1): track 9.19 -> 18.4 mm
- net Net-(J9-Pad2): track 0.00 -> 6.24 mm
- net Net-(J1-Pad1): track 5.25 -> 10.5 mm
- net Net-(C7-Pad1): track 4.86 -> 9.72 mm
- net Net-(J5-Pad1): track 3.45 -> 6.89 mm
- net Net-(C1-Pad1): track 2.80 -> 5.59 mm
- net Net-(C5-Pad1): track 0.00 -> 1.73 mm
Other:
- board size 17.1 x 12.4 mm -> 38.1 x 39.9 mm
